Commit message: Update arm.urdf

File: subprocesses/arm/kinematics/arm.urdf (robot description, URDF)
Before this commit: robot simple_arm, 8 links, 7 joints
Links:
- removed link base
- added link base_link
Joints:
- joint J1: parent base -> base_link

Commit message: Update arm.urdf (bro chatgpt gave it to me using mm as units smh)

File: subprocesses/arm/kinematics/arm.urdf (robot description, URDF)
Before this commit: robot simple_arm, 8 links, 7 joints
Joints:
- joint J2: origin xyz=0 0 20 rpy=0 0 0 -> xyz=0 0 0.020 rpy=0 0 0
- joint J3: origin xyz=0 0 400 rpy=0 0 0 -> xyz=0 0 0.400 rpy=0 0 0
- joint J4: origin xyz=0 0 400 rpy=0 0 0 -> xyz=0 0 0.400 rpy=0 0 0
- joint J5: origin xyz=0 0 20 rpy=0 0 0 -> xyz=0 0 0.020 rpy=0 0 0
- joint J6: origin xyz=0 0 20 rpy=0 0 0 -> xyz=0 0 0.020 rpy=0 0 0
- joint ee_fixed: origin xyz=0 0 20 rpy=0 0 0 -> xyz=0 0 0.020 rpy=0 0 0
